Commit message: agregar cassis

File: description/robot_core.xacro (robot description, xacro)
@@ -1,10 +1,22 @@
 <?xml version="1.0"?>
 <robot xmlns:xacro="http://www.ros.org/wiki/xacro"  >
+    <material name="white">
+        <color rgba="1 1 1 1" />
+    </material>
+    <material name="orange">
+        <color rgba="1 0.3 0.1 1" />
+    </material>
+    <material name="blue">
+        <color rgba="0.2 0.2 1 1" />
+    </material>
+    <material name="black">
+        <color rgba="0 0 0 1" />
+    </material>
     <!-- base -->
     <link name="base_link"></link>
-    <join name="chassis_joint" type="fix">
+    <join name="chassis_joint" type="fixed">
         <parent link="base_link"/>
         <child link="chassis"/>
-        <origen xyz="0.1 0 0"/>
+        <origin xyz="-0.1 0 0"/>
     </join>
     <link name="chassis">
@@ -14,4 +26,5 @@
                 <box size="0.3 0.3 0.15"/>
             </geometry>
+            <material name="white"/>
         </visual>
     </link>

Commit message: corregir baselink-chassis link

File: description/robot_core.xacro (robot description, xacro)
@@ -13,19 +13,12 @@
         <color rgba="0 0 0 1" />
     </material>
-    <!-- base -->
-    <link name="base_link"></link>
-    <join name="chassis_joint" type="fixed">
+    <!-- BASE LINK -->
+    <link name="base_link"> </link>
+    <!-- CHASSIS LINK -->
+    <joint name="chassis_joint" type="fixed">
         <parent link="base_link"/>
         <child link="chassis"/>
         <origin xyz="-0.1 0 0"/>
-    </join>
-    <link name="chassis">
-        <visual>
-            <origin xyz="0.15 0 0.075"/>
-            <geometry>
-                <box size="0.3 0.3 0.15"/>
-            </geometry>
-            <material name="white"/>
-        </visual>
-    </link>
+    </joint>
+    <link name="chassis"></link>
 </robot>

Commit message: carro como esta en el tuto

File: description/robot_core.xacro (robot description, xacro)
@@ -21,4 +21,58 @@
         <origin xyz="-0.1 0 0"/>
     </joint>
-    <link name="chassis"></link>
+    <link name="chassis">
+        <visual>
+            <origin xyz="0.15 0 0.075"/>
+            <geometry>
+                <box size="0.3 0.3 0.15"/>
+            </geometry>
+            <material name="white"/>
+        </visual>
+        <collision>
+            <origin xyz="0.15 0 0.075"/>
+            <geometry>
+                <box size="0.3 0.3 0.15"/>
+            </geometry>
+        </collision>
+    </link>
+    <!-- LEFT WHEEL LINK -->
+    <joint name="left_wheel_joint" type="continuous">
+        <parent link="base_link"/>
+        <child link="left_wheel"/>
+        <origin xyz="0 0.175 0" rpy="-${pi/2} 0 0" />
+        <axis xyz="0 0 1"/>
+    </joint>
+    <link name="left_wheel">
+        <visual>
+            <geometry>
+                <cylinder radius="0.05" length="0.04"/>
+            </geometry>
+            <material name="blue"/>
+        </visual>
+        <collision>
+            <geometry>
+                <cylinder radius="0.05" length="0.04"/>
+            </geometry>
+        </collision>
+    </link>
+    <!-- RIGHT WHEEL LINK -->
+    <joint name="right_wheel_joint" type="continuous">
+        <parent link="base_link"/>
+        <child link="right_wheel"/>
+        <origin xyz="0 -0.175 0" rpy="${pi/2} 0 0" />
+        <axis xyz="0 0 -1"/>
+    </joint>
+    <link name="right_wheel">
+        <visual>
+            <geometry>
+                <cylinder radius="0.05" length="0.04"/>
+            </geometry>
+            <material name="blue"/>
+        </visual>
+        <collision>
+            <geometry>
+                <cylinder radius="0.05" length="0.04"/>
+            </geometry>
+        </collision>
+    </link>
 </robot>

Commit message: cuatro ruedas

File: description/robot_core.xacro (robot description, xacro)
@@ -36,12 +36,12 @@
         </collision>
     </link>
-    <!-- LEFT WHEEL LINK -->
-    <joint name="left_wheel_joint" type="continuous">
+    <!-- BOTTOM LEFT WHEEL LINK -->
+    <joint name="Bottom_left_wheel_joint" type="continuous">
         <parent link="base_link"/>
-        <child link="left_wheel"/>
+        <child link="Bottom_left_wheel"/>
         <origin xyz="0 0.175 0" rpy="-${pi/2} 0 0" />
         <axis xyz="0 0 1"/>
     </joint>
-    <link name="left_wheel">
+    <link name="Bottom_left_wheel">
         <visual>
             <geometry>
@@ -56,12 +56,52 @@
         </collision>
     </link>
-    <!-- RIGHT WHEEL LINK -->
-    <joint name="right_wheel_joint" type="continuous">
+    <!-- BOTTOM RIGHT WHEEL LINK -->
+    <joint name="Bottom_right_wheel_joint" type="continuous">
         <parent link="base_link"/>
-        <child link="right_wheel"/>
+        <child link="Bottom_right_wheel"/>
         <origin xyz="0 -0.175 0" rpy="${pi/2} 0 0" />
         <axis xyz="0 0 -1"/>
     </joint>
-    <link name="right_wheel">
+    <link name="Bottom_right_wheel">
+        <visual>
+            <geometry>
+                <cylinder radius="0.05" length="0.04"/>
+            </geometry>
+            <material name="blue"/>
+        </visual>
+        <collision>
+            <geometry>
+                <cylinder radius="0.05" length="0.04"/>
+            </geometry>
+        </collision>
+    </link>
+    <!-- TOP LEFT WHEEL LINK -->
+    <joint name="Top_left_wheel_joint" type="continuous">
+        <parent link="base_link"/>
+        <child link="Top_left_wheel"/>
+        <origin xyz="0.175 0.175 0" rpy="-${pi/2} 0 0" />
+        <axis xyz="0 0 1"/>
+    </joint>
+    <link name="Top_left_wheel">
+        <visual>
+            <geometry>
+                <cylinder radius="0.05" length="0.04"/>
+            </geometry>
+            <material name="blue"/>
+        </visual>
+        <collision>
+            <geometry>
+                <cylinder radius="0.05" length="0.04"/>
+            </geometry>
+        </collision>
+    </link>
+    <!-- TOP RIGHT WHEEL LINK -->
+    <joint name="Top_right_wheel_joint" type="continuous">
+        <parent link="base_link"/>
+        <child link="Top_right_wheel"/>
+        <origin xyz="0.175 -0.175 0" rpy="${pi/2} 0 0" />
+        <axis xyz="0 0 -1"/>
+    </joint>
+    <link name="Top_right_wheel">
         <visual>
             <geometry>

Commit message: Agregar inercias y el luncher.py

File: description/robot_core.xacro (robot description, xacro)
@@ -1,4 +1,5 @@
 <?xml version="1.0"?>
 <robot xmlns:xacro="http://www.ros.org/wiki/xacro"  >
+    <xacro:include filename="inertial_macros.xacro"/>
     <material name="white">
         <color rgba="1 1 1 1" />
@@ -35,4 +36,7 @@
             </geometry>
         </collision>
+        <xacro:inertial_box mass="0.5" x="0.3" y="0.3" z="0.15">
+            <origin xyz="0.15 0 0.075" rpy="0 0 0"/>
+        </xacro:inertial_box>
     </link>
     <!-- BOTTOM LEFT WHEEL LINK -->
@@ -55,4 +59,7 @@
             </geometry>
         </collision>
+        <xacro:inertial_cylinder mass="0.1" length="0.04" radius="0.05">
+            <origin xyz="0 0 0" rpy="0 0 0"/>
+        </xacro:inertial_cylinder>
     </link>
     <!-- BOTTOM RIGHT WHEEL LINK -->
@@ -75,4 +82,7 @@
             </geometry>
         </collision>
+        <xacro:inertial_cylinder mass="0.1" length="0.04" radius="0.05">
+            <origin xyz="0 0 0" rpy="0 0 0"/>
+        </xacro:inertial_cylinder>
     </link>
     <!-- TOP LEFT WHEEL LINK -->
@@ -95,4 +105,7 @@
             </geometry>
         </collision>
+        <xacro:inertial_cylinder mass="0.1" length="0.04" radius="0.05">
+            <origin xyz="0 0 0" rpy="0 0 0"/>
+        </xacro:inertial_cylinder>
     </link>
     <!-- TOP RIGHT WHEEL LINK -->
@@ -115,4 +128,7 @@
             </geometry>
         </collision>
+        <xacro:inertial_cylinder mass="0.1" length="0.04" radius="0.05">
+            <origin xyz="0 0 0" rpy="0 0 0"/>
+        </xacro:inertial_cylinder>
     </link>
 </robot>

Commit message: Corregir colores Gazebo

File: description/robot_core.xacro (robot description, xacro)
@@ -40,4 +40,7 @@
         </xacro:inertial_box>
     </link>
+    <gazebo reference="chassis">
+        <material>Gazebo/White</material>
+    </gazebo>
     <!-- BOTTOM LEFT WHEEL LINK -->
     <joint name="Bottom_left_wheel_joint" type="continuous">
@@ -63,4 +66,7 @@
         </xacro:inertial_cylinder>
     </link>
+    <gazebo reference="Bottom_left_wheel">
+        <material>Gazebo/Blue</material>
+    </gazebo>
     <!-- BOTTOM RIGHT WHEEL LINK -->
     <joint name="Bottom_right_wheel_joint" type="continuous">
@@ -86,4 +92,7 @@
         </xacro:inertial_cylinder>
     </link>
+    <gazebo reference="Bottom_right_wheel">
+        <material>Gazebo/Blue</material>
+    </gazebo>
     <!-- TOP LEFT WHEEL LINK -->
     <joint name="Top_left_wheel_joint" type="continuous">
@@ -109,4 +118,7 @@
         </xacro:inertial_cylinder>
     </link>
+    <gazebo reference="Top_left_wheel">
+        <material>Gazebo/Orange</material>
+    </gazebo>
     <!-- TOP RIGHT WHEEL LINK -->
     <joint name="Top_right_wheel_joint" type="continuous">
@@ -132,3 +144,6 @@
         </xacro:inertial_cylinder>
     </link>
+    <gazebo reference="Top_right_wheel">
+        <material>Gazebo/Orange</material>
+    </gazebo>
 </robot>
